Commit message: CV course presentation last commit

File: racecar_description/urdf/racecar.xacro (robot description, xacro)
@@ -185,4 +185,20 @@
     <parent link="chassis"/>
     <child link="base_imu_link"/>
+  </joint>
+ <!-- Basler_camera config -->
+  <link name="base_basler_camera_link">
+    <visual>
+      <origin xyz="0 0 0" rpy="0 0 0"/>
+      <geometry>
+        <box size="0.0293 0.029 0.029"/>
+      </geometry>
+      <material name="gray"/>
+    </visual>
+  </link>
+   <joint name="base_basler_camera_joint" type="fixed">
+    <axis xyz="0 0 0" />
+    <origin xyz="0.145 0.0 0.208" rpy="0 0 0"/>
+    <parent link="chassis"/>
+    <child link="base_basler_camera_link"/>
   </joint>
 <!-- full zed camera config -->

Commit message: test SLAM systems

File: racecar_description/urdf/racecar.xacro (robot description, xacro)
@@ -191,14 +191,31 @@
       <origin xyz="0 0 0" rpy="0 0 0"/>
       <geometry>
-        <box size="0.0293 0.029 0.029"/>
-      </geometry>
-      <material name="gray"/>
-    </visual>
-  </link>
-   <joint name="base_basler_camera_joint" type="fixed">
+        <box size="0.033 0.029 0.029"/>
+      </geometry>
+      <material name="orange"/>
+    </visual>
+  </link>
+  <joint name="base_basler_camera_joint" type="fixed">
     <axis xyz="0 0 0" />
-    <origin xyz="0.145 0.0 0.208" rpy="0 0 0"/>
+    <origin xyz="0.145 0.0 0.218" rpy="0 0 0"/>
     <parent link="chassis"/>
     <child link="base_basler_camera_link"/>
+  </joint>
+  <link name="base_basler_camera_lens_link">
+    <visual>
+      <origin xyz="0 0 0" rpy="0 1.57 0"/>
+      <geometry>
+         <cylinder length="0.033" radius="0.0140"/>
+      </geometry>
+      <material name="dark_grey">
+                <color rgba="0.1 0.1 0.1 1"/>
+      </material>
+    </visual>
+  </link>
+  <joint name="base_basler_camera_lens_joint" type="fixed">
+    <axis xyz="0 0 0" />
+    <origin xyz="0.033 0 0" rpy="0 0 0"/>
+    <parent link="base_basler_camera_link"/>
+    <child link="base_basler_camera_lens_link"/>
   </joint>
 <!-- full zed camera config -->
